Commit message: fixing urdf

File: ma_robo/urdf/robo.xacro (robot description, xacro)
@@ -255,10 +255,10 @@
   <parent link="base_link"/>
   <child link="arm_mount_link"/>
-  <origin xyz="0 0 ${base_height/2}" rpy="0 0 0"/>
+  <origin xyz="-0.035 0 ${base_height/2}" rpy="0 0 0"/>
 </joint>
 <joint name="arm_to_robot_joint" type="fixed">
   <parent link="arm_mount_link"/>
   <child link="arm_base_link"/>
-  <origin xyz="0 0 0.02" rpy="0 0 1.57"/>
+  <origin xyz="0 0 0.011" rpy="0 0 1.57"/>
 </joint>
 </robot>

File: ma_robo/urdf/so_100_arm.urdf (robot description, URDF)
Before this commit: robot so_100_arm, 8 links, 7 joints
Links:
- link Base: geometry collision mesh filename=package://ma_robo/models/so_100_arm_5dof/meshes/Base.STL; visual mesh filename=package://ma_robo/models/so_100_arm_5dof/meshes/Base.STL
- link Fixed_Gripper: geometry collision mesh filename=package://ma_robo/models/so_100_arm_5dof/meshes/Fixed_Gripp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; visual mesh filename=package://ma_robo/models/so_100_arm_5dof/meshes/Fixed_Gripp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
- link Lower_Arm: geometry collision mesh filename=package://ma_robo/models/so_100_arm_5dof/meshes/Lower_Arm.S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; visual mesh filename=package://ma_robo/models/so_100_arm_5dof/meshes/Lower_Arm.S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
- link Moving_Jaw: geometry collision mesh filename=package://ma_robo/models/so_100_arm_5dof/meshes/Moving_Jaw.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; visual mesh filename=package://ma_robo/models/so_100_arm_5dof/meshes/Moving_Jaw.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
- link Shoulder_Rotation_Pitch: geometry collision mesh filename=package://ma_robo/models/so_100_arm_5dof/meshes/Shoulder_Ro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; visual mesh filename=package://ma_robo/models/so_100_arm_5dof/meshes/Shoulder_Ro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
- link Upper_Arm: geometry collision mesh filename=package://ma_robo/models/so_100_arm_5dof/meshes/Upper_Arm.S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; visual mesh filename=package://ma_robo/models/so_100_arm_5dof/meshes/Upper_Arm.S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
- link Wrist_Pitch_Roll: geometry collision mesh filename=package://ma_robo/models/so_100_arm_5dof/meshes/Wrist_Pitch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; visual mesh filename=package://ma_robo/models/so_100_arm_5dof/meshes/Wrist_Pitch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
